File: pcb/tesina.kicad_pcb (KiCad board)
At the start: 2 copper layers, 70 x 35 mm, 48 parts, among them J1 Conn_01x02_Male, J2 Conn_01x02_Male, J5 AMP2_IN, J6 AMP3_IN, J7 AMP2_OUT, J8 AMP3_OUT, Q1 BFP640, Q3 BFP640, U1 Single_Stub_Input, U2 Single_Stub_Output

Commit message: design finished
Parts:
- removed C10, C8: 100nF, Capacitor_SMD:C_1206_3216Metric
- moved R7 5.81 mm to (115.6, 96.7)
- moved R6 5.72 mm to (114.0, 96.7)
- moved R5 4.82 mm to (125.7, 96.6), turned to -90 degrees
- moved R3 4.80 mm to (87.2, 98.2)
- moved R4 4.63 mm to (87.2, 99.8)
- moved J2 3.62 mm to (123.7, 102.0)
- moved R1 3.23 mm to (109.7, 96.7), turned to -90 degrees
- moved R8 3.18 mm to (87.2, 101.5)
- moved L3 2.87 mm to (100.9, 95.1)
- moved C6 2.49 mm to (123.7, 97.5), turned to 90 degrees
- moved C4 2.35 mm to (87.2, 96.5)
- moved R2 1.97 mm to (121.5, 96.6)
- moved C3 1.80 mm to (111.8, 97.5), turned to 90 degrees
- moved R12 1.71 mm to (139.2, 92.7)
- moved R11 1.58 mm to (139.2, 94.3)
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Routing:
- net /Amplifier2/VCC: track 15.3 -> 32.9 mm
- net /Amplifier2/VCC2: track 20.8 -> 30.4 mm
- net /Amplifier1/RF1_OUT_BF: track 11.4 -> 3.58 mm
- net /Amplifier1/VCC2: track 24.8 -> 30.1 mm
- net /Amplifier1/DC1_2: track 13.8 -> 10.7 mm
- net Net-(J2-Pad1): track 2.91 -> 5.06 mm
- net /Amplifier1/VCC: track 33.8 -> 35.9 mm
- net Net-(J1-Pad1): track 2.89 -> 4.89 mm
- net /Amplifier2/RF2_IN_AM: track 2.48 -> 3.85 mm
- net /Amplifier1/RF1_IN_AM: track 3.30 -> 2.11 mm
- net /Amplifier1/DC1_1: track 19.1 -> 20.1 mm
- net Net-(C3-Pad2): track 5.60 -> 6.56 mm
- net /DC: track 7.04 -> 6.44 mm
- net GND: vias 76 -> 66
- added copper zone on F.Cu, net /Amplifier1/RF1_IN_AM
- added copper zone on F.Cu, net /Amplifier1/RF1_IN_BM
- added copper zone on F.Cu, net /Amplifier1/RF1_OUT_BF
- added copper zone on F.Cu, net /Amplifier2/RF2_IN_AM
- added copper zone on F.Cu, net /Amplifier2/RF2_OUT_BM

Commit message: PCB ready for review
Parts:
- removed C11: 100nF, Capacitor_SMD:C_1206_3216Metric
- removed C19: 398fF, Capacitor_SMD:C_0603_1608Metric
- removed L11: 1.26nH, Nicobigio01:Coilcraft_0906-xxLx
- added C8: 11.8pF, Capacitor_SMD:C_0603_1608Metric, F.Cu at (132.8, 84.4)
- added L2: 2.55nH, Nicobigio01:Coilcraft_0906-xxLx, F.Cu at (143.1, 86.0)
- L15: value 1.78nH -> 7.15 nH; footprint Nicobigio01:Coilcraft_0906-xxLx -> Nicobigio01:Coilcraft_mod
- U1: footprint Nicobigio01:Microwave_Single_Stub_Input -> Nicobigio01:Microwave_Stub_In2
- U2: footprint Nicobigio01:Microwave_SIngle_Stub_Output -> Nicobigio01:Microwave_Stub_Out2
- moved R8 30.6 mm to (117.1, 94.8)
- moved C4 29.9 mm to (117.1, 96.5)
- moved R3 29.9 mm to (117.1, 98.1)
- moved R4 29.9 mm to (117.1, 99.8)
- moved U2 18.3 mm to (102.1, 102.9), turned to 0 degrees
- moved H4 16.8 mm to (86.8, 97.8)
- moved C3 14.9 mm to (126.7, 98.5)
- moved C6 14.9 mm to (138.6, 98.5)
- moved J1 14.9 mm to (126.7, 103.1)
- moved R1 14.9 mm to (124.6, 97.7)
- moved R5 14.9 mm to (140.5, 97.7)
- moved R6 14.9 mm to (128.8, 97.7)
- moved R9 14.9 mm to (134.8, 97.7)
- moved J2 14.9 mm to (138.5, 103.1)
- moved R2 14.9 mm to (136.4, 97.7)
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Connections:
- net /Amplifier2/STAGE2_OUT renamed /Amplifier2/RF2_OUT
- C20 pad 1: Net-(C19-Pad2) -> Net-(C20-Pad1)
- L15 pad 1: Net-(C19-Pad2) -> /Amplifier2/RF2_OUT_BM
- L3 pad 1: /Amplifier1/RF1_OUT_BF -> /Amplifier1/RF1_OUT_AM
Routing:
- net /Amplifier1/DC1_2: track 10.7 -> 57.1 mm
- net /Amplifier2/VCC: track 32.9 -> 4.26 mm
- net /Amplifier2/VCC2: track 30.4 -> 5.34 mm
- net /Amplifier1/RF1_OUT_AM: track 3.33 -> 26.7 mm
- net /Amplifier1/VCC2: track 30.1 -> 12.6 mm
- net /Amplifier1/DC1_1: track 20.1 -> 6.28 mm
- net /Amplifier1/RF1_IN_AM: track 2.11 -> 14.0 mm
- net /Amplifier1/VCC: track 35.9 -> 27.2 mm
- net Net-(C19-Pad2): track 4.26 -> 0.00 mm
- net Net-(C20-Pad1): track 0.00 -> 4.04 mm
- net /Amplifier2/RF2_OUT_BM: track 5.50 -> 9.35 mm
- net /Amplifier1/RF1_OUT_BF: track 3.58 -> 0.00 mm
- net Net-(C16-Pad1): track 16.3 -> 12.9 mm
- net /Amplifier1/RF1_IN_BM: track 6.30 -> 3.01 mm
- net Net-(C7-Pad2): track 8.60 -> 10.4 mm
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- removed copper zone on F.Cu, net /Amplifier1/RF1_IN_AM
- removed copper zone on F.Cu, net /Amplifier2/RF2_OUT_BM
