File: pcb/tesina.kicad_pcb (KiCad board)
At the start: 2 copper layers, 70 x 35 mm, 45 parts, among them J1 Conn_01x02_Male, J2 Conn_01x02_Male, J5 AMP2_IN, J6 AMP3_IN, J7 AMP2_OUT, J8 AMP3_OUT, Q1 BFP640, Q3 BFP640, U1 Single_Stub_Input, U2 Single_Stub_Output

Commit message: cleanup
Parts:
- moved C4 20.6 mm to (96.6, 94.7), turned to 90 degrees
- moved L3 14.2 mm to (98.9, 99.0), turned to 90 degrees
- moved R8 1.71 mm to (117.1, 96.5)
Connections:
- net /Amplifier1/RF1_IN renamed /Amplifier1/STAGE1_IN
- net /Amplifier1/RF1_OUT renamed /Amplifier1/STAGE2_OUT
- net /Amplifier2/RF2_IN renamed /Amplifier2/STAGE1_IN
- net /Amplifier2/RF2_OUT renamed /Amplifier2/STAGE2_OUT
- net Net-(C16-Pad1) renamed /Amplifier2/DC2_2
- net Net-(C7-Pad2) renamed /Amplifier2/RF2_IN_BM
- L3 pad 1: /Amplifier1/RF1_OUT_AM -> /Amplifier1/RF1_OUT_BF
Routing:
- net /Amplifier1/DC1_1: track 6.28 -> 52.2 mm, vias 0 -> 2
- net /Amplifier1/DC1_2: track 57.1 -> 83.7 mm
- net /Amplifier1/RF1_OUT_BF: track 0.00 -> 3.20 mm
- net /Amplifier1/RF1_OUT_AM: track 26.7 -> 24.7 mm
- net /Amplifier2/RF2_IN_BM: track 10.4 -> 9.39 mm
- net /Amplifier1/VCC2: track 12.6 -> 13.4 mm
- removed copper zone on F.Cu, net /Amplifier1/RF1_IN_BM
Other:
- board text removed: "-Come vanno condensatori -cambia qualcosa dc prima o dopo -metal loss e come ottenere tan delta a temp -din o iso fori -attenzione condensatori metric ecc."
- board text removed: "filtro grosso pad alimentazione alimentazione anche negativa condenatore parallelo filtro piccolo cambiare fori massa transistor"
