File: pcb/amp1.kicad_sch (KiCad schematic)
At the start: 14 parts, among them Q1 BFP640, U1 Single_Stub_Input, U2 Single_Stub_Output

Commit message: design finished
Parts:
- removed C10, C8: 100nF, Capacitor_SMD:C_1206_3216Metric, symbol Device:C
Changed lines of the file:
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@@
 (kicad_sch (version 20211123) (generator eeschema)
   (paper "A4")
-  (junction (at 160.02 88.9) (diameter 0) (color 0 0 0 0)
-  )
   (junction (at 153.67 88.9) (diameter 0) (color 0 0 0 0)
   )
@@
   (junction (at 139.7 88.9) (diameter 0) (color 0 0 0 0)
   )
-  (junction (at 96.52 88.9) (diameter 0) (color 0 0 0 0)
-  )
   (wire (pts (xy 153.67 97.79) (xy 153.67 99.06))
     (stroke (width 0) (type default) (color 0 0 0 0))
@@
     (stroke (width 0) (type default) (color 0 0 0 0))
   )
-  (wire (pts (xy 160.02 74.93) (xy 160.02 73.66))
-    (stroke (width 0) (type default) (color 0 0 0 0))
-  )
   (wire (pts (xy 111.76 88.9) (xy 139.7 88.9))
     (stroke (width 0) (type default) (color 0 0 0 0))
   )
-  (wire (pts (xy 96.52 97.79) (xy 96.52 99.06))
-    (stroke (width 0) (type default) (color 0 0 0 0))
-  )
   (wire (pts (xy 154.94 114.3) (xy 153.67 114.3))
     (stroke (width 0) (type default) (color 0 0 0 0))
@@
     (stroke (width 0) (type default) (color 0 0 0 0))
   )
-  (wire (pts (xy 96.52 88.9) (xy 111.76 88.9))
+  (wire (pts (xy 95.25 88.9) (xy 111.76 88.9))
     (stroke (width 0) (type default) (color 0 0 0 0))
   )
@@
     (stroke (width 0) (type default) (color 0 0 0 0))
   )
-  (wire (pts (xy 95.25 88.9) (xy 96.52 88.9))
-    (stroke (width 0) (type default) (color 0 0 0 0))
-  )
   (wire (pts (xy 153.67 77.47) (xy 153.67 80.01))
     (stroke (width 0) (type default) (color 0 0 0 0))
   )
-  (wire (pts (xy 96.52 90.17) (xy 96.52 88.9))
-    (stroke (width 0) (type default) (color 0 0 0 0))
-  )
   (wire (pts (xy 111.76 90.17) (xy 111.76 88.9))
     (stroke (width 0) (type default) (color 0 0 0 0))
@@
     (stroke (width 0) (type default) (color 0 0 0 0))
   )
-  (wire (pts (xy 160.02 88.9) (xy 161.29 88.9))
+  (wire (pts (xy 153.67 88.9) (xy 161.29 88.9))
     (stroke (width 0) (type default) (color 0 0 0 0))
   )
@@
   )
   (wire (pts (xy 153.67 99.06) (xy 153.67 100.33))
-    (stroke (width 0) (type default) (color 0 0 0 0))
-  )
-  (wire (pts (xy 153.67 88.9) (xy 160.02 88.9))
-    (stroke (width 0) (type default) (color 0 0 0 0))
-  )
-  (wire (pts (xy 160.02 82.55) (xy 160.02 88.9))
     (stroke (width 0) (type default) (color 0 0 0 0))
   )
@@
   (hierarchical_label "VCC" (shape input) (at 153.67 77.47 90)
     (effects (font (size 1.27 1.27)) (justify left))
-  )
-  (symbol (lib_id "Device:C") (at 96.52 93.98 0) (mirror y) (unit 1)
-    (in_bom yes) (on_board yes)
-    (property "Reference" "C8" (id 0) (at 90.17 93.98 0)
-      (effects (font (size 1.27 1.27)) (justify right))
-    )
-    (property "Value" "100nF" (id 1) (at 90.17 96.52 0)
-      (effects (font (size 1.27 1.27)) (justify right))
-    )
-    (property "Footprint" "Capacitor_SMD:C_1206_3216Metric" (id 2) (at 95.5548 97.79 0)
-      (effects (font (size 1.27 1.27)) hide)
-    )
-    (property "Datasheet" "~" (id 3) (at 96.52 93.98 0)
-      (effects (font (size 1.27 1.27)) hide)
-    )
-    (pin "1")
-    (pin "2")
   )
   (symbol (lib_id "Device:C") (at 111.76 93.98 0) (mirror y) (unit 1)
@@
     (pin "2")
   )
-  (symbol (lib_id "power:GND") (at 160.02 73.66 180) (unit 1)
-    (in_bom yes) (on_board yes) (fields_autoplaced)
-    (property "Reference" "#PWR0112" (id 0) (at 160.02 67.31 0)
-      (effects (font (size 1.27 1.27)) hide)
-    )
-    (property "Value" "GND" (id 1) (at 160.02 68.58 0))
-    (property "Footprint" "" (id 2) (at 160.02 73.66 0)
-      (effects (font (size 1.27 1.27)) hide)
-    )
-    (property "Datasheet" "" (id 3) (at 160.02 73.66 0)
-      (effects (font (size 1.27 1.27)) hide)
-    )
-    (pin "1")
-  )
   (symbol (lib_id "power:GND") (at 170.18 91.44 0) (unit 1)
     (in_bom yes) (on_board yes)
@@
     (pin "2")
   )
-  (symbol (lib_id "Device:C") (at 160.02 78.74 0) (mirror x) (unit 1)
-    (in_bom yes) (on_board yes)
-    (property "Reference" "C10" (id 0) (at 166.37 78.74 0)
-      (effects (font (size 1.27 1.27)) (justify right))
-    )
-    (property "Value" "100nF" (id 1) (at 166.37 76.2 0)
-      (effects (font (size 1.27 1.27)) (justify right))
-    )
-    (property "Footprint" "Capacitor_SMD:C_1206_3216Metric" (id 2) (at 160.9852 74.93 0)
-      (effects (font (size 1.27 1.27)) hide)
-    )
-    (property "Datasheet" "~" (id 3) (at 160.02 78.74 0)
-      (effects (font (size 1.27 1.27)) hide)
-    )
-    (pin "1")
-    (pin "2")
-  )
   (symbol (lib_id "power:GND") (at 154.94 128.27 0) (unit 1)
     (in_bom yes) (on_board yes) (fields_autoplaced)
@@
     (pin "2")
   )
-  (symbol (lib_id "power:GND") (at 96.52 99.06 0) (unit 1)
-    (in_bom yes) (on_board yes) (fields_autoplaced)
-    (property "Reference" "#PWR0113" (id 0) (at 96.52 105.41 0)
-      (effects (font (size 1.27 1.27)) hide)
-    )
-    (property "Value" "GND" (id 1) (at 96.52 104.14 0))
-    (property "Footprint" "" (id 2) (at 96.52 99.06 0)
-      (effects (font (size 1.27 1.27)) hide)
-    )
-    (property "Datasheet" "" (id 3) (at 96.52 99.06 0)
-      (effects (font (size 1.27 1.27)) hide)
-    )
-    (pin "1")
-  )
   (symbol (lib_id "power:GND") (at 111.76 99.06 0) (unit 1)

Commit message: PCB ready for review
Parts:
- U1: footprint Nicobigio01:Microwave_Single_Stub_Input -> Nicobigio01:Microwave_Stub_In2
- U2: footprint Nicobigio01:Microwave_SIngle_Stub_Output -> Nicobigio01:Microwave_Stub_Out2
Connections:
- net RF1_OUT_AM: now also L3.1
- net RF1_OUT_BF: no longer L3.1
Changed lines of the file:
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@@
   (junction (at 153.67 88.9) (diameter 0) (color 0 0 0 0)
   )
-  (junction (at 153.67 99.06) (diameter 0) (color 0 0 0 0)
+  (junction (at 180.34 99.06) (diameter 0) (color 0 0 0 0)
   )
   (junction (at 154.94 114.3) (diameter 0) (color 0 0 0 0)
@@
   (junction (at 139.7 88.9) (diameter 0) (color 0 0 0 0)
   )
-  (wire (pts (xy 153.67 97.79) (xy 153.67 99.06))
-    (stroke (width 0) (type default) (color 0 0 0 0))
-  )
   (wire (pts (xy 198.12 99.06) (xy 208.28 99.06))
     (stroke (width 0) (type default) (color 0 0 0 0))
@@
     (stroke (width 0) (type default) (color 0 0 0 0))
   )
+  (wire (pts (xy 153.67 97.79) (xy 180.34 97.79))
+    (stroke (width 0) (type default) (color 0 0 0 0))
+  )
   (wire (pts (xy 156.21 113.03) (xy 156.21 114.3))
     (stroke (width 0) (type default) (color 0 0 0 0))
@@
     (stroke (width 0) (type default) (color 0 0 0 0))
   )
-  (wire (pts (xy 176.53 99.06) (xy 190.5 99.06))
+  (wire (pts (xy 176.53 99.06) (xy 180.34 99.06))
     (stroke (width 0) (type default) (color 0 0 0 0))
   )
@@
     (stroke (width 0) (type default) (color 0 0 0 0))
   )
+  (wire (pts (xy 180.34 99.06) (xy 190.5 99.06))
+    (stroke (width 0) (type default) (color 0 0 0 0))
+  )
   (wire (pts (xy 153.67 99.06) (xy 153.67 100.33))
+    (stroke (width 0) (type default) (color 0 0 0 0))
+  )
+  (wire (pts (xy 180.34 97.79) (xy 180.34 99.06))
     (stroke (width 0) (type default) (color 0 0 0 0))
   )
@@
     (property "Reference" "U2" (id 0) (at 170.18 107.95 0))
     (property "Value" "Single_Stub_Output" (id 1) (at 171.45 111.76 0))
-    (property "Footprint" "Nicobigio01:Microwave_SIngle_Stub_Output" (id 2) (at 168.91 96.52 0)
+    (property "Footprint" "Nicobigio01:Microwave_Stub_Out2" (id 2) (at 168.91 96.52 0)
       (effects (font (size 1.27 1.27)) hide)
     )
@@
     (property "Reference" "U1" (id 0) (at 123.19 99.06 0))
     (property "Value" "Single_Stub_Input" (id 1) (at 120.65 101.6 0))
-    (property "Footprint" "Nicobigio01:Microwave_Single_Stub_Input" (id 2) (at 131.445 106.68 0)
-      (effects (font (size 1.27 1.27)) hide)
-    )
+    (property "Footprint" "Nicobigio01:Microwave_Stub_In2" (id 2) (at 131.445 106.68 0)
+      (effects (font (size 1.27 1.27)) hide)
+    )

Commit message: cleanup
Connections:
- net RF1_OUT_AM: no longer L3.1
- net RF1_OUT_BF: now also L3.1
Other:
- note added: "Il valore di lambda nel simbolo e' sbagliato, nella scheda la lunghezza e' quella giusta pero'"

Commit message: graduated
Parts:
- R3: value 44kΩ -> 43kΩ
- R4: value 375Ω -> 390Ω
- R8: value Ω -> 43kΩ
- U1: footprint Nicobigio01:Microwave_Stub_In2 -> Nicobigio01:Microwave_Single_Stub_Input
- U2: footprint Nicobigio01:Microwave_Stub_Out2 -> Nicobigio01:Microwave_SIngle_Stub_Output
Other:
- note removed: "Il valore di lambda nel simbolo e' sbagliato, nella scheda la lunghezza e' quella giusta pero'"
- moved on the sheet: C1, C2, C4, L1, L3, R3, R4, R8, U1
